File: Hardware/BOSS-Coll-Interface/2021-05-03 Coll-Interface.sch (EAGLE design)
At the start: 5 parts, among them J1 Amphenol 75869-330LF, J2 TE_1-2834016-2, X1 TE 5747835-4

Commit message: Changed hole size on capacitor leads
Other:
- note added: "C1 Holes for leads too small"
Changed lines of the file:
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@@
 <sheet>
 <plain>
+<text x="73.66" y="45.72" size="1.778" layer="250">C1 Holes for leads too small</text>
 </plain>
 <instances>
