File: Hardware/BOSS-Coll-Interface/Coll-Interface.sch (EAGLE design)
At the start: 5 parts, among them J1 Amphenol 75869-330LF, J2 TE_1-2834016-2, X1 TE 5747835-4

Commit message: Changed hole size on capacitor leads
Other:
- note added: "C1 Holes for leads were too small; Updated on 2021-05-22"
Changed lines of the file:
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@@
 <part name="X1" library="AUmlib" library_urn="urn:adsk.eagle:library:9166017" deviceset="DE-37-TE-CONNECTIVITY-5747835-4" device="" package3d_urn="urn:adsk.eagle:package:28471019/2" value="TE 5747835-4"/>
 <part name="J2" library="AUmlib" library_urn="urn:adsk.eagle:library:9166017" deviceset="TERMINAL_BLOCK_2PIN_1-2834016-2" device="" package3d_urn="urn:adsk.eagle:package:27672122/2" value="TE_1-2834016-2"/>
-<part name="C1" library="AUmlib" library_urn="urn:adsk.eagle:library:9166017" deviceset="ELECTROLYTIC_UHE1H471MHD3" device="" package3d_urn="urn:adsk.eagle:package:27672260/2" value="UHE1H471MHD3"/>
+<part name="C1" library="AUmlib" library_urn="urn:adsk.eagle:library:9166017" deviceset="ELECTROLYTIC_UHE1H471MHD3" device="" package3d_urn="urn:adsk.eagle:package:27672260/3" value="UHE1H471MHD3"/>
 <part name="D1" library="AUmlib" library_urn="urn:adsk.eagle:library:9166017" deviceset="SCHOTTKY-PMEG6030EVPX" device="" package3d_urn="urn:adsk.eagle:package:28188986/2"/>
 </parts>
@@
 <sheet>
 <plain>
+<text x="73.66" y="43.18" size="1.778" layer="250">C1 Holes for leads were too small;
+Updated on 2021-05-22</text>
 </plain>
 <instances>
@@
 </drawing>
 <compatibility>
+<note version="6.3" minversion="6.2.2" severity="warning">
+Since Version 6.2.2 text objects can contain more than one line,
+which will not be processed correctly with this version.
+</note>
 <note version="8.2" severity="warning">
 Since Version 8.2, EAGLE supports online libraries. The ids
